Commit message: [Dev] add ros2_controller

File: description/lidar.xacro (robot description, xacro)
@@ -1,11 +1,11 @@
 <?xml version="1.0"?>
-<robot xmlns:xacro="http://www.ros.org/wiki/xacro"  name="robot">
-<joint name="laser_joint" type="fixed">
-    <parent link="chassis"/>
-    <child link="laser_frame"/>
-    <origin xyz="0.1 0 0.175" rpy="0.0 0.0 0.0"/>
-</joint>
-<link name="laser_frame">
-     <visual>
+<robot xmlns:xacro="http://www.ros.org/wiki/xacro" >
+    <joint name="laser_joint" type="fixed">
+        <parent link="chassis"/>
+        <child link="laser_frame"/>
+        <origin xyz="0.1 0 0.175" rpy="0 0 0"/>
+    </joint>
+    <link name="laser_frame">
+        <visual>
             <geometry>
                 <cylinder radius="0.05" length="0.04"/>
@@ -21,6 +21,6 @@
             <origin xyz="0 0 0" rpy="0 0 0"/>
         </xacro:inertial_cylinder>
-</link>
-<gazebo reference="laser_frame">
+    </link>
+    <gazebo reference="laser_frame">
         <material>Gazebo/Red</material>
         <sensor name="laser" type="ray">

File: description/robot.urdf.xacro (robot description, xacro)
@@ -1,7 +1,8 @@
 <?xml version="1.0"?>
 <robot xmlns:xacro="http://www.ros.org/wiki/xacro"  name="robot">
-    <xacro:include filename="robot_core.xacro" />
-    <xacro:include filename="gazebo_control.xacro" />
+   <xacro:include filename="robot_core.xacro" />
+  <xacro:include filename="ros2_control.xacro" />
+   <!--  <xacro:include filename="gazebo_control.xacro" />-->
     <xacro:include filename="lidar.xacro" />
-<xacro:include filename="depth_camera.xacro" />
+<xacro:include filename="camera.xacro" />
 </robot>
